File: elec/layouts/default/default.kicad_pcb (KiCad board)
At the start: 2 copper layers, 72.5 x 31 mm, 10 parts

Commit message: feat: completed and ordered
Parts:
- J3, J4: footprint ScrewTerminal_2.54_3P:TerminalBlock_Phoenix_MPT-0,5-3-2.54_1x03_P2.54mm_Horizontal -> KF141R_3P:KF141R_3P
Routing:
- net 23: track 0.00 -> 149.0 mm
- net gnd: track 147.9 -> 0.00 mm, vias 85 -> 0
- net 25: track 0.00 -> 108.8 mm, vias 0 -> 1
- net 1: track 107.3 -> 0.00 mm, vias 2 -> 0
- net vcc_5v: track 66.4 -> 0.00 mm, vias 1 -> 0
- net 24: track 0.00 -> 66.2 mm, vias 0 -> 1
- removed copper zone on B.Cu, net gnd
- removed copper zone on F.Cu, net gnd
Other:
- board size 72.5 x 31 mm -> 75 x 31 mm
- board text removed: "configure 12V before mounting"
